File: cad/touchboard/touchboard.kicad_pcb (KiCad board)
At the start: 2 copper layers, 170.1 x 84.1 mm, 34 parts, among them J1 Conn_01x02, J2 Conn_01x02, J8 Conn_01x02, U2 LM2596, U3 ESP32-DEVKIT-V1, U4 adafruit-MAX98357, U5 adafruit-MAX98357

Commit message: designed pcb
Parts:
- added C4: 10u, Capacitor_THT:CP_Radial_D4.0mm_P1.50mm, F.Cu at (176.0, 58.5)
- added C5: 100n, Capacitor_THT:C_Disc_D3.8mm_W2.6mm_P2.50mm, F.Cu at (181.0, 57.5)
- added C6: CFA1, Capacitor_THT:CP_Radial_D4.0mm_P1.50mm, F.Cu at (173.5, 91.0)
- added C7: CFA2, Capacitor_THT:C_Disc_D3.8mm_W2.6mm_P2.50mm, F.Cu at (175.5, 97.0)
- added C8: CFA1, Capacitor_THT:CP_Radial_D4.0mm_P1.50mm, F.Cu at (178.5, 91.0)
- added C9: CFA2, Capacitor_THT:C_Disc_D3.8mm_W2.6mm_P2.50mm, F.Cu at (181.5, 96.0)
- added D4: LED, LED_THT:LED_D3.0mm, F.Cu at (192.0, 46.0)
- added J3: Conn_01x02, Connector_Phoenix_MSTB:PhoenixContact_MSTBA_2,5_2-G_1x02_P5.00mm_Horizontal, F.Cu at (199.2, 52.5)
- added J4: Conn_01x04, Connector_JST:JST_EH_B4B-EH-A_1x04_P2.50mm_Vertical, F.Cu at (176.2, 101.0)
- added JP2: SolderJumper_3_Bridged12, Jumper:SolderJumper-3_P1.3mm_Bridged12_RoundedPad1.0x1.5mm, F.Cu at (188.0, 86.7)
- added Q1: PN2222A, Package_TO_SOT_THT:TO-92_Inline, F.Cu at (180.0, 66.0)
- added Q2: PN2222A, Package_TO_SOT_THT:TO-92_Inline, F.Cu at (187.0, 66.3)
- added Q3: IRLZ44N, Package_TO_SOT_THT:TO-220-3_Vertical, F.Cu at (200.5, 64.0)
- added R2: 10k, Resistor_THT:R_Axial_DIN0207_L6.3mm_D2.5mm_P7.62mm_Horizontal, F.Cu at (160.2, 68.0)
- added R3: 10k, Resistor_THT:R_Axial_DIN0207_L6.3mm_D2.5mm_P7.62mm_Horizontal, F.Cu at (191.8, 60.0)
- added R4: 10k, Resistor_THT:R_Axial_DIN0207_L6.3mm_D2.5mm_P7.62mm_Horizontal, F.Cu at (195.0, 56.2)
- added R5: 470, Resistor_THT:R_Axial_DIN0207_L6.3mm_D2.5mm_P7.62mm_Horizontal, F.Cu at (188.0, 53.8)
- added R7: RFA, Resistor_THT:R_Axial_DIN0207_L6.3mm_D2.5mm_P7.62mm_Horizontal, F.Cu at (168.2, 87.0)
- added R8: RFA, Resistor_THT:R_Axial_DIN0207_L6.3mm_D2.5mm_P7.62mm_Horizontal, F.Cu at (167.2, 83.0)
- added RG1: 100, Resistor_THT:R_Axial_DIN0207_L6.3mm_D2.5mm_P7.62mm_Horizontal, F.Cu at (180.1, 79.4)
- added RSD1: 47k, Resistor_THT:R_Axial_DIN0207_L6.3mm_D2.5mm_P7.62mm_Horizontal, F.Cu at (180.1, 75.4)
- moved C32 79.1 mm to (82.0, 99.5), turned to -90 degrees
- moved D2 50.3 mm to (166.9, 53.0), turned to 0 degrees
- moved R1 43.4 mm to (163.0, 50.2), turned to -90 degrees
- moved C35 36.1 mm to (135.5, 83.0)
- moved C34 29.5 mm to (131.0, 82.5), turned to -90 degrees
- moved J8 24.4 mm to (166.5, 101.0)
- moved C33 24.3 mm to (143.0, 81.0), turned to -90 degrees
- moved D3 23.8 mm to (161.5, 101.0), turned to 180 degrees
- moved D1 17.1 mm to (138.6, 69.0), turned to 180 degrees
- moved R6 12.3 mm to (160.2, 92.0)
- moved R10 12.3 mm to (160.2, 96.0)
- moved J1 7.07 mm to (181.5, 53.8)
- moved J2 7.07 mm to (167.5, 46.0)
- moved U1 6.00 mm to (140.4, 88.1)
- moved C1 5.92 mm to (167.3, 62.0), turned to 0 degrees
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Connections:
- C1 pad 2: GNDA -> GND
- J1 pad 1: GNDA -> GND
- U2 pad 2: GNDA -> GND
- U3 pad 20: unconnected-(U3-D35-Pad20) -> POT_GAIN
- U3 pad 21: unconnected-(U3-D32-Pad21) -> BCLK
- U3 pad 22: unconnected-(U3-D33-Pad22) -> LRC
- U3 pad 23: unconnected-(U3-D25-Pad23) -> DAC1
- U3 pad 24: unconnected-(U3-D26-Pad24) -> DAC2
- U3 pad 25: unconnected-(U3-D27-Pad25) -> DIN
- U3 pad 5: unconnected-(U3-D4-Pad5) -> LED_PWM1
- U4 pad 1: unconnected-(U4-Vin-Pad1) -> +5V
- U4 pad 3: unconnected-(U4-~{SD_MODE}-Pad3) -> Net-(U4-~{SD_MODE})
- U4 pad 4: unconnected-(U4-GAIN-Pad4) -> GAIN
- U4 pad 5: unconnected-(U4-DIN-Pad5) -> DIN
- U4 pad 6: unconnected-(U4-BCLK-Pad6) -> BCLK
- U4 pad 7: unconnected-(U4-LRC-Pad7) -> LRC
- U5 pad 1: unconnected-(U5-Vin-Pad1) -> +5V
- U5 pad 3: unconnected-(U5-~{SD_MODE}-Pad3) -> +5V
- U5 pad 4: unconnected-(U5-GAIN-Pad4) -> GAIN
- U5 pad 5: unconnected-(U5-DIN-Pad5) -> DIN
- U5 pad 6: unconnected-(U5-BCLK-Pad6) -> BCLK
- U5 pad 7: unconnected-(U5-LRC-Pad7) -> LRC
Routing:
- net +3.3V: track 0.00 -> 197.2 mm
- net +5V: track 0.00 -> 193.7 mm
- net DIN: track 0.00 -> 121.8 mm, vias 0 -> 1
- net BCLK: track 0.00 -> 116.7 mm, vias 0 -> 1
- net LRC: track 0.00 -> 91.3 mm, vias 0 -> 1
- net I2C_SDA: track 0.00 -> 82.2 mm
- net +12V: track 0.00 -> 80.6 mm
- net I2C_SCL: track 0.00 -> 75.0 mm
- net ELE11: track 0.00 -> 69.2 mm
- net ELE0: track 0.00 -> 65.2 mm
- net ELE10: track 0.00 -> 57.6 mm
- net ELE1: track 0.00 -> 54.2 mm
- net ELE9: track 0.00 -> 46.9 mm
- net ELE2: track 0.00 -> 43.2 mm
- net VSPI_CS: track 0.00 -> 42.4 mm
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Other:
- board size 170.1 x 84.1 mm -> 170.1 x 90.1 mm

Commit message: pcb done
Parts:
- added H1: MountingHole, MountingHole:MountingHole_3.2mm_M3, F.Cu at (46.0, 107.0)
- added H2: MountingHole, MountingHole:MountingHole_3.2mm_M3, F.Cu at (206.0, 107.0)
- added J5: Conn_01x03, Connector_JST:JST_EH_B3B-EH-A_1x03_P2.50mm_Vertical, F.Cu at (148.0, 101.0)
- added JP1: Jumper_3_Open, Connector_PinHeader_2.54mm:PinHeader_1x03_P2.54mm_Vertical, F.Cu at (188.0, 90.0)
- added JP3: Jumper_3_Open, Connector_PinHeader_2.54mm:PinHeader_1x03_P2.54mm_Vertical, F.Cu at (52.0, 120.5)
- added U7: ~, SD:SD_module, F.Cu at (146.7, 83.8)
- E1, E10, E11, E12, E2, E3, E4, E5, E6, E7, E8, E9: footprint Connector_Audio:Jack_3.5mm_CUI_SJ1-3523N_Horizontal -> Connector_Audio:Jack_3.5mm_CUI_SJ-3523-SMT_Horizontal
- JP2: value SolderJumper_3_Bridged12 -> Jumper_3_Open; footprint Jumper:SolderJumper-3_P1.3mm_Bridged12_RoundedPad1.0x1.5mm -> Connector_PinHeader_2.54mm:PinHeader_1x03_P2.54mm_Vertical
- moved JP2 145.9 mm to (46.0, 120.5), turned to 180 degrees
- moved E1 12.0 mm to (61.0, 120.0), turned to 180 degrees
- moved E12 10.2 mm to (192.9, 120.0), turned to 180 degrees
- moved E2 10.0 mm to (73.0, 120.0), turned to 180 degrees
- moved D3 8.60 mm to (170.0, 102.5), turned to 90 degrees
- moved E11 8.06 mm to (180.9, 120.0), turned to 180 degrees
- moved E3 8.06 mm to (85.0, 120.0), turned to 180 degrees
- moved R2 8.06 mm to (152.2, 67.0)
- moved R1 8.00 mm to (163.0, 58.2)
- moved R10 6.90 mm to (165.8, 92.0), turned to 180 degrees
- moved E10 6.08 mm to (169.0, 120.0), turned to 180 degrees
- moved E4 6.08 mm to (97.0, 120.0), turned to 180 degrees
- moved C2 6.00 mm to (114.0, 61.0), turned to 180 degrees
- moved J8 6.00 mm to (160.5, 101.0)
- moved R6 4.56 mm to (158.0, 96.0)
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Connections:
- E1 pad R: +3.3V -> SVCC
- E1 pad S: GND -> SGND
- E10 pad R: +3.3V -> SVCC
- E10 pad S: GND -> SGND
- E11 pad R: +3.3V -> SVCC
- E11 pad S: GND -> SGND
- E12 pad R: +3.3V -> SVCC
- E12 pad S: GND -> SGND
- E2 pad R: +3.3V -> SVCC
- E2 pad S: GND -> SGND
- E3 pad R: +3.3V -> SVCC
- E3 pad S: GND -> SGND
- E4 pad R: +3.3V -> SVCC
- E4 pad S: GND -> SGND
- E5 pad R: +3.3V -> SVCC
- E5 pad S: GND -> SGND
- E6 pad R: +3.3V -> SVCC
- E6 pad S: GND -> SGND
- E7 pad R: +3.3V -> SVCC
- E7 pad S: GND -> SGND
- E8 pad R: +3.3V -> SVCC
- E8 pad S: GND -> SGND
- E9 pad R: +3.3V -> SVCC
- E9 pad S: GND -> SGND
- JP2 pad 1: +5V -> GND
- JP2 pad 2: GAIN -> SGND
- JP2 pad 3: Net-(JP2-B) -> unconnected-(JP2-B-Pad3)
- RG1 pad 2: Net-(JP2-B) -> Net-(JP1-B)
- U3 pad 19: unconnected-(U3-D34-Pad19) -> BTN1
Routing:
- net SGND: track 0.00 -> 155.4 mm
- net SVCC: track 0.00 -> 142.8 mm
- net GND: track 0.00 -> 93.5 mm, vias 0 -> 15
- net +3.3V: track 197.2 -> 290.6 mm
- net HSPI_CS: track 0.00 -> 90.7 mm
- net HSPI_MISO: track 0.00 -> 86.0 mm, vias 0 -> 1
- net HSPI_CLK: track 0.00 -> 84.5 mm, vias 0 -> 1
- net HSPI_MOSI: track 0.00 -> 78.5 mm, vias 0 -> 1
- net BTN1: track 11.6 -> 81.6 mm
- net LED_PWM1: track 17.3 -> 87.1 mm
- net POT_GAIN: track 0.00 -> 62.8 mm
- net DAC1: track 16.2 -> 71.1 mm, vias 0 -> 1
- net DAC2: track 17.8 -> 65.4 mm, vias 0 -> 1
- net LRC: track 91.3 -> 116.8 mm, vias 1 -> 2
- net +5V: track 193.7 -> 209.7 mm, vias 0 -> 1
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- added copper zone on B.Cu, net GND
- added copper zone on F.Cu, net GND
Other:
- board size 170.1 x 90.1 mm -> 170 x 90 mm
- board text added: "BTN"
- board text added: "DAC"
- board text added: "POT"

Commit message: pcb board update
Parts:
- U4, U5: value adafruit-MAX98357 -> MAX98357
- moved H1 2.00 mm to (46.0, 109.0)
- moved H2 2.00 mm to (206.0, 109.0)
Routing:
- net GND: vias 15 -> 26
Other:
- board text added: "TOUCHBOARD V1.0"

Commit message: touchboard pcb cad v1 finished
Parts:
- U4, U5: value MAX98357 -> adafruit-MAX98357
- moved C32 0.50 mm to (82.0, 100.0)
Connections:
- U1 pad 2: unconnected-(U1-IRQ-Pad2) -> IRQ
- U3 pad 5: LED_PWM1 -> IRQ
- U3 pad 7: unconnected-(U3-TX2-Pad7) -> LED_PWM1
Routing:
- net IRQ: track 0.00 -> 96.1 mm
- net GND: track 93.5 -> 23.0 mm, vias 26 -> 30
- net +3.3V: track 290.6 -> 232.8 mm
- net LED_PWM1: track 87.1 -> 92.2 mm
- net I2C_SDA: track 82.2 -> 78.7 mm
- net DIN: track 123.7 -> 126.9 mm
- net I2C_SCL: track 75.0 -> 72.5 mm
- net +5V: track 209.7 -> 212.2 mm
- net DAC2: track 65.4 -> 66.6 mm
- net HSPI_MISO: track 86.0 -> 86.9 mm
- net VSPI_MOSI: track 31.6 -> 32.3 mm
- net ELE6: track 11.9 -> 12.4 mm
