File: cad/touchboard/touchboard.kicad_sch (KiCad schematic)
At the start: 34 parts, among them J1 Conn_01x02, J2 Conn_01x02, J8 Conn_01x02, U2 LM2596, U3 ESP32-DEVKIT-V1, U4 adafruit-MAX98357, U5 adafruit-MAX98357

Commit message: designed pcb
Parts:
- added C4: 10u, Capacitor_THT:CP_Radial_D4.0mm_P1.50mm, symbol Device:C_Polarized
- added C5: 100n, Capacitor_THT:C_Disc_D3.8mm_W2.6mm_P2.50mm, symbol Device:C
- added C6, C8: CFA1, Capacitor_THT:CP_Radial_D4.0mm_P1.50mm, symbol Device:C
- added C7, C9: CFA2, Capacitor_THT:C_Disc_D3.8mm_W2.6mm_P2.50mm, symbol Device:C
- added D4: LED, LED_THT:LED_D3.0mm, symbol Device:LED
- added J3: Conn_01x02, Connector_Phoenix_MSTB:PhoenixContact_MSTBA_2,5_2-G_1x02_P5.00mm_Horizontal, symbol Connector_Generic:Conn_01x02
- added J4: Conn_01x04, Connector_JST:JST_EH_B4B-EH-A_1x04_P2.50mm_Vertical, symbol Connector_Generic:Conn_01x04
- added JP2: SolderJumper_3_Bridged12, Jumper:SolderJumper-3_P1.3mm_Bridged12_RoundedPad1.0x1.5mm, symbol Jumper:SolderJumper_3_Bridged12
- added Q1, Q2: PN2222A, Package_TO_SOT_THT:TO-92_Inline, symbol Transistor_BJT:PN2222A
- added Q3: IRLZ44N, Package_TO_SOT_THT:TO-220-3_Vertical, symbol Transistor_FET:IRLZ44N
- added R2, R3, R4: 10k, Resistor_THT:R_Axial_DIN0207_L6.3mm_D2.5mm_P7.62mm_Horizontal, symbol Device:R
- added R5: 470, Resistor_THT:R_Axial_DIN0207_L6.3mm_D2.5mm_P7.62mm_Horizontal, symbol Device:R
- added R7, R8: RFA, Resistor_THT:R_Axial_DIN0207_L6.3mm_D2.5mm_P7.62mm_Horizontal, symbol Device:R
- added RG1: 100, Resistor_THT:R_Axial_DIN0207_L6.3mm_D2.5mm_P7.62mm_Horizontal, symbol Device:R
- added RSD1: 47k, Resistor_THT:R_Axial_DIN0207_L6.3mm_D2.5mm_P7.62mm_Horizontal, symbol Device:R
Connections:
- net GNDA is gone; now on net GND: C1.2, J1.1 (Pin_1), U2.2 (GND)
- net +12V: now also C4.1, C5.1, D4.2 (A), J3.1 (Pin_1), R3.1, R4.1
- net +5V: now also U4.1 (Vin), U5.1 (Vin), U5.3 (~{SD_MODE}), JP2.1 (A), RSD1.1
- net GND: now also C4.2, C5.2, C6.2, C7.2, C8.2, C9.2, J4.2 (Pin_2), J4.4 (Pin_4), Q1.1 (E), Q2.1 (E), Q3.3 (S), RG1.1
- net GAIN: now reaches U5.4 (GAIN)
- net GAIN: now also U4.4 (GAIN), JP2.2 (C)
- net DIN: now reaches U5.5 (DIN)
- net DIN: now also U3.25 (D27), U4.5 (DIN)
- net BCLK: now reaches U5.6 (BCLK)
- net BCLK: now also U3.21 (D32), U4.6 (BCLK)
- net LRC: now reaches U5.7 (LRC)
- net LRC: now also U3.22 (D33), U4.7 (LRC)
- net at U4.3 (~{SD_MODE}): now also RSD1.2
- net POT_GAIN: now reaches U3.20 (D35)
- net DAC1: now reaches U3.23 (D25)
- net DAC1: now also R7.1
- net DAC2: now reaches U3.24 (D26)
- net DAC2: now also R8.1
- net LED_PWM1: now reaches U3.5 (D4)
- net LED_PWM1: now also R2.1
- new net: J3.2 (Pin_2), Q3.2 (D), R5.1
- new net: C8.1, C9.1, J4.3 (Pin_3), R8.2
- new net: Q1.2 (B), R2.2
- new net: Q1.3 (C), Q2.2 (B), R3.2
- new net: Q2.3 (C), Q3.1 (G), R4.2
- new net: JP2.3 (B), RG1.2
- new net: C6.1, C7.1, J4.1 (Pin_1), R7.2
- new net: D4.1 (K), R5.2
Other:
- moved on the sheet: C32, U3, U4, U5, U6

Commit message: pcb done
Parts:
- removed JP2: SolderJumper_3_Bridged12, Jumper:SolderJumper-3_P1.3mm_Bridged12_RoundedPad1.0x1.5mm, symbol Jumper:SolderJumper_3_Bridged12
- added H1, H2: MountingHole, MountingHole:MountingHole_3.2mm_M3, symbol Mechanical:MountingHole
- added J5: Conn_01x03, Connector_JST:JST_EH_B3B-EH-A_1x03_P2.50mm_Vertical, symbol Connector_Generic:Conn_01x03
- added JP1, JP2, JP3: Jumper_3_Open, Connector_PinHeader_2.54mm:PinHeader_1x03_P2.54mm_Vertical, symbol Jumper:Jumper_3_Open
- added U7: ~, SD:SD_module, symbol SD_module:SD_module
- E1, E10, E11, E12, E2, E3, E4, E5, E6, E7, E8, E9: footprint Connector_Audio:Jack_3.5mm_CUI_SJ1-3523N_Horizontal -> Connector_Audio:Jack_3.5mm_CUI_SJ-3523-SMT_Horizontal
Connections:
- net +3.3V: now also J5.1 (Pin_1), JP3.1 (A); no longer E1.R, E10.R, E11.R, E12.R, E2.R, E3.R, E4.R, E5.R, E6.R, E7.R, E8.R, E9.R
- net +5V: now also JP1.1 (A), U7.5 (VCC)
- net BTN1: now also U3.19 (D34)
- net GAIN: now also JP1.2 (C)
- net GND: now also J5.3 (Pin_3), JP2.1 (A), U7.6 (GND); no longer E1.S, E10.S, E11.S, E12.S, E2.S, E3.S, E4.S, E5.S, E6.S, E7.S, E8.S, E9.S
- net HSPI_CLK: now also U7.2 (SCK)
- net HSPI_CS: now also U7.1 (CS)
- net HSPI_MISO: now also U7.4 (MISO)
- net HSPI_MOSI: now also U7.3 (MOSI)
- net POT_GAIN: now also J5.2 (Pin_2)
- net at RG1.2: now also JP1.3 (B)
- new net SGND: E1.S, E10.S, E11.S, E12.S, E2.S, E3.S, E4.S, E5.S, E6.S, E7.S, E8.S, E9.S, JP2.2 (C)
- new net SVCC: E1.R, E10.R, E11.R, E12.R, E2.R, E3.R, E4.R, E5.R, E6.R, E7.R, E8.R, E9.R, JP3.2 (C)

Commit message: touchboard pcb cad v1 finished
Connections:
- net LED_PWM1: now also U3.7 (TX2); no longer U3.5 (D4)
- net IRQ: now reaches U1.2 (IRQ)
- net IRQ: now also U3.5 (D4)
